File: platform16.kicad_sch (KiCad schematic)
At the start: 108 parts, among them CN1 PJ-342, CN2 PJ-342, CN3 PJ-342, IC1 PAM8908JER, J2 Conn_01x03, J4 SM03B-SRSS-TB, Q1 SS8050, Q3 SS8050, SW2 TS-1095PS-A165B2-C3D2, SW3 TS-1095PS-A165B2-C3D2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

Commit message: tweaks
Parts:
- added TP1, TP2: TestPoint, TestPoint:TestPoint_THTPad_D4.0mm_Drill2.0mm, symbol Connector:TestPoint
- R24, R25, R27, R33: LCSC C25792 -> C11702
- R26, R28, R30, R32: LCSC C25792 -> C25744
- R37: LCSC C11702 -> C25744
- RV1, RV10, RV11, RV12, RV13, RV14, RV15, RV16, RV2, RV3, RV4, RV5, RV6, RV7, RV8, RV9: LCSC C470305 -> C470448
Connections:
- net +3V3: now also TP1.1
- net GND: now also TP2.1

Commit message: another iteration
Parts:
- added TP3, TP4: TestPoint, TestPoint:TestPoint_THTPad_D4.0mm_Drill2.0mm, symbol Connector:TestPoint
- RV1, RV10, RV11, RV12, RV13, RV14, RV15, RV16, RV2, RV3, RV4, RV5, RV6, RV7, RV8, RV9: LCSC C470448 -> C470449
- TP1, TP2: now not fitted; now left out of the parts list
Connections:
- net LINE_L: now also TP3.1
- net LINE_R: now also TP4.1
Other:
- note removed: "TODO: button, switch, addressable LED?"
Changed lines of the file:
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@@
 	)
 	(junction
+		(at 370.84 48.26)
+		(diameter 0)
+		(color 0 0 0 0)
+	)
+	(junction
 		(at 201.93 21.59)
 		(diameter 0)
@@
 	)
 	(junction
+		(at 381 50.8)
+		(diameter 0)
+		(color 0 0 0 0)
+	)
+	(junction
 		(at 300.99 101.6)
 		(diameter 0)
@@
 		)
 	)
-	(text "TODO: button, switch, addressable LED?"
-		(exclude_from_sim no)
-		(at 286.258 161.544 0)
-		(effects
-			(font
-				(size 1.27 1.27)
-			)
-		)
-	)
 	(text "12MHz Crystal"
 		(exclude_from_sim no)
@@
 			)
 		)
-		(property "LCSC" "C470448"
+		(property "LCSC" "C470449"
 			(at 312.42 196.85 0)
 			(effects
@@
 			)
 		)
-		(property "LCSC" "C470448"
+		(property "LCSC" "C470449"
 			(at 340.36 234.95 0)
 			(effects
@@
 			)
 		)
-		(property "LCSC" "C470448"
+		(property "LCSC" "C470449"
 			(at 298.45 196.85 0)
 			(effects
@@
 			)
 		)
-		(property "LCSC" "C470448"
+		(property "LCSC" "C470449"
 			(at 312.42 209.55 0)
 			(effects
@@
 		(unit 1)
 		(exclude_from_sim no)
-		(in_bom yes)
+		(in_bom no)
 		(on_board yes)
-		(dnp no)
+		(dnp yes)
 		(fields_autoplaced yes)
 		(property "Reference" "TP2"
@@
 	)
 	(symbol
+		(lib_id "Connector:TestPoint")
+		(at 381 50.8 0)
+		(unit 1)
+		(exclude_from_sim no)
+		(in_bom no)
+		(on_board yes)
+		(dnp yes)
+		(fields_autoplaced yes)
+		(property "Reference" "TP4"
+			(at 383.54 46.2279 0)
+			(effects
+				(font
+					(size 1.27 1.27)
+				)
+				(justify left)
+			)
+		)
+		(property "Value" "TestPoint"
+			(at 383.54 48.7679 0)
+			(effects
+				(font
+					(size 1.27 1.27)
+				)
+				(justify left)
+			)
+		)
+		(property "Footprint" "TestPoint:TestPoint_THTPad_D4.0mm_Drill2.0mm"
+			(at 386.08 50.8 0)
+			(effects
+				(font
+					(size 1.27 1.27)
+				)
+				(hide yes)
+			)
+		)
+		(property "Datasheet" "~"
+			(at 386.08 50.8 0)
+			(effects
+				(font
+					(size 1.27 1.27)
+				)
+				(hide yes)
+			)
+		)
+		(property "Description" "test point"
+			(at 381 50.8 0)
+			(effects
+				(font
+					(size 1.27 1.27)
+				)
+				(hide yes)
+			)
+		)
+		(property "Label" "LINE R"
+			(at 381 50.8 0)
+			(effects
+				(font
+					(size 1.27 1.27)
+				)
+				(hide yes)
+			)
+		)
+		(pin "1"
+		)
+		(instances
+			(project "platform16"
+				(path "/8ea573ca-1d7e-409c-bbf9-736989e92912"
+					(reference "TP4")
+					(unit 1)
+				)
+			)
+		)
+	)
+	(symbol
 		(lib_id "Device:R")
 		(at 151.13 119.38 90)
@@
 			)
 		)
-		(property "LCSC" "C470448"
+		(property "LCSC" "C470449"
 			(at 326.39 209.55 0)
 			(effects
@@
 			)
 		)
-		(property "LCSC" "C470448"
+		(property "LCSC" "C470449"
 			(at 298.45 234.95 0)
 			(effects
@@
 			)
 		)
-		(property "LCSC" "C470448"
+		(property "LCSC" "C470449"
 			(at 340.36 222.25 0)
 			(effects
@@
 			)
 		)
-		(property "LCSC" "C470448"
+		(property "LCSC" "C470449"
 			(at 326.39 196.85 0)
 			(effects
@@
 			)
 		)
-		(property "LCSC" "C470448"
+		(property "LCSC" "C470449"
 			(at 312.42 222.25 0)
 			(effects
@@
 			)
 		)
-		(property "LCSC" "C470448"
+		(property "LCSC" "C470449"
 			(at 312.42 234.95 0)
 			(effects
@@
 			)
 		)
-		(property "LCSC" "C470448"
+		(property "LCSC" "C470449"
 			(at 340.36 209.55 0)
 			(effects
@@
 			)
 		)
-		(property "LCSC" "C470448"
+		(property "LCSC" "C470449"
 			(at 326.39 234.95 0)
 			(effects
@@
 			)
 		)
-		(property "LCSC" "C470448"
+		(property "LCSC" "C470449"
 			(at 326.39 222.25 0)
 			(effects
@@
 	)
 	(symbol
+		(lib_id "Connector:TestPoint")
+		(at 370.84 48.26 0)
+		(unit 1)
+		(exclude_from_sim no)
+		(in_bom no)
+		(on_board yes)
+		(dnp yes)
+		(fields_autoplaced yes)
+		(property "Reference" "TP3"
+			(at 373.38 43.6879 0)
+			(effects
+				(font
+					(size 1.27 1.27)
+				)
+				(justify left)
+			)
+		)
+		(property "Value" "TestPoint"
+			(at 373.38 46.2279 0)
+			(effects
+				(font
+					(size 1.27 1.27)
+				)
+				(justify left)
+			)
+		)
+		(property "Footprint" "TestPoint:TestPoint_THTPad_D4.0mm_Drill2.0mm"
+			(at 375.92 48.26 0)
+			(effects
+				(font
+					(size 1.27 1.27)
+				)
+				(hide yes)
+			)
+		)
+		(property "Datasheet" "~"
+			(at 375.92 48.26 0)
+			(effects
+				(font
+					(size 1.27 1.27)
+				)
+				(hide yes)
+			)
+		)
+		(property "Description" "test point"
+			(at 370.84 48.26 0)
+			(effects
+				(font
+					(size 1.27 1.27)
+				)
+				(hide yes)
+			)
+		)
+		(property "Label" "LINE L"
+			(at 370.84 48.26 0)
+			(effects
+				(font
+					(size 1.27 1.27)
+				)
+				(hide yes)
+			)
+		)
+		(pin "1"
+		)
+		(instances
+			(project "platform16"
+				(path "/8ea573ca-1d7e-409c-bbf9-736989e92912"
+					(reference "TP3")
+					(unit 1)
+				)
+			)
+		)
+	)
+	(symbol
 		(lib_id "Device:R_Small")
 		(at 238.76 254 0)
@@
 			)
 		)
-		(property "LCSC" "C470448"
+		(property "LCSC" "C470449"
 			(at 298.45 222.25 0)
 			(effects
@@
 			)
 		)
-		(property "LCSC" "C470448"
+		(property "LCSC" "C470449"
 			(at 298.45 209.55 0)
 			(effects
@@
 		(unit 1)
 		(exclude_from_sim no)
-		(in_bom yes)
+		(in_bom no)
 		(on_board yes)
-		(dnp no)
+		(dnp yes)
 		(fields_autoplaced yes)
 		(property "Reference" "TP1"
@@
 			)
 		)
-		(property "LCSC" "C470448"
+		(property "LCSC" "C470449"
 			(at 340.36 196.85 0)
 			(effects

Commit message: potentiometer tweaks
Parts:
- RV1, RV10, RV11, RV12, RV13, RV14, RV15, RV16, RV2, RV3, RV4, RV5, RV6, RV7, RV8, RV9: LCSC C470449 -> C470305
Changed lines of the file:
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@@
 			)
 		)
-		(property "LCSC" "C470449"
+		(property "LCSC" "C470305"
 			(at 312.42 196.85 0)
 			(effects
@@
 			)
 		)
-		(property "LCSC" "C470449"
+		(property "LCSC" "C470305"
 			(at 340.36 234.95 0)
 			(effects
@@
 			)
 		)
-		(property "LCSC" "C470449"
+		(property "LCSC" "C470305"
 			(at 298.45 196.85 0)
 			(effects
@@
 			)
 		)
-		(property "LCSC" "C470449"
+		(property "LCSC" "C470305"
 			(at 312.42 209.55 0)
 			(effects
@@
 			)
 		)
-		(property "LCSC" "C470449"
+		(property "LCSC" "C470305"
 			(at 326.39 209.55 0)
 			(effects
@@
 			)
 		)
-		(property "LCSC" "C470449"
+		(property "LCSC" "C470305"
 			(at 298.45 234.95 0)
 			(effects
@@
 			)
 		)
-		(property "LCSC" "C470449"
+		(property "LCSC" "C470305"
 			(at 340.36 222.25 0)
 			(effects
@@
 			)
 		)
-		(property "LCSC" "C470449"
+		(property "LCSC" "C470305"
 			(at 326.39 196.85 0)
 			(effects
@@
 			)
 		)
-		(property "LCSC" "C470449"
+		(property "LCSC" "C470305"
 			(at 312.42 222.25 0)
 			(effects
@@
 			)
 		)
-		(property "LCSC" "C470449"
+		(property "LCSC" "C470305"
 			(at 312.42 234.95 0)
 			(effects
@@
 			)
 		)
-		(property "LCSC" "C470449"
+		(property "LCSC" "C470305"
 			(at 340.36 209.55 0)
 			(effects
@@
 			)
 		)
-		(property "LCSC" "C470449"
+		(property "LCSC" "C470305"
 			(at 326.39 234.95 0)
 			(effects
@@
 			)
 		)
-		(property "LCSC" "C470449"
+		(property "LCSC" "C470305"
 			(at 326.39 222.25 0)
 			(effects
@@
 			)
 		)
-		(property "LCSC" "C470449"
+		(property "LCSC" "C470305"
 			(at 298.45 222.25 0)
 			(effects
@@
 			)
 		)
-		(property "LCSC" "C470449"
+		(property "LCSC" "C470305"
 			(at 298.45 209.55 0)
 			(effects
@@
 			)
 		)
-		(property "LCSC" "C470449"
+		(property "LCSC" "C470305"
 			(at 340.36 196.85 0)
 			(effects

Commit message: basic readme
Parts:
- SW2, SW3: LCSC C3010220 -> C782843
Changed lines of the file:
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@@
 (kicad_sch
-	(version 20231120)
+	(version 20250114)
 	(generator "eeschema")
-	(generator_version "8.0")
+	(generator_version "9.0")
 	(paper "A3")
+	(circle
+		(center 142.24 135.255)
+		(radius 0.635)
+		(stroke
+			(width 0)
+			(type default)
+			(color 132 0 0 1)
+		)
+		(fill
+			(type color)
+			(color 132 0 0 1)
+		)
+	)
+	(text "CPVDD"
+		(exclude_from_sim no)
+		(at 386.842 24.384 0)
+		(effects
+			(font
+				(size 1.27 1.27)
+			)
+		)
+	)
+	(text "JST Debug Connector"
+		(exclude_from_sim no)
+		(at 37.465 183.515 0)
+		(effects
+			(font
+				(size 1.27 1.27)
+			)
+			(justify left bottom)
+		)
+	)
+	(text "For Opposite Side"
+		(exclude_from_sim no)
+		(at 90.678 62.23 0)
+		(effects
+			(font
+				(size 1.27 1.27)
+			)
+		)
+	)
+	(text "16 Pots"
+		(exclude_from_sim no)
+		(at 308.864 187.706 0)
+		(effects
+			(font
+				(size 2.54 2.54)
+			)
+			(justify left bottom)
+		)
+	)
+	(text "USB"
+		(exclude_from_sim no)
+		(at 18.542 85.852 0)
+		(effects
+			(font
+				(size 2.54 2.54)
+			)
+			(justify left bottom)
+		)
+	)
+	(text "Clock In\n"
+		(exclude_from_sim no)
+		(at 109.982 251.968 0)
+		(effects
+			(font
+				(size 2.54 2.54)
+			)
+			(justify left bottom)
+		)
+	)
+	(text "AMPLIFIER"
+		(exclude_from_sim no)
+		(at 177.546 27.432 0)
+		(effects
+			(font
+				(size 2.54 2.54)
+			)
+		)
+	)
+	(text "AVDD\n"
+		(exclude_from_sim no)
+		(at 349.758 24.638 0)
+		(effects
+			(font
+				(size 1.27 1.27)
+			)
+		)
+	)
+	(text "TODO: reduce the gain so it is safe for headphones?\nOr just trust that users will reduce volume from line level?"
+		(exclude_from_sim no)
+		(at 146.812 84.074 0)
+		(effects
+			(font
+				(size 1.27 1.27)
+			)
+		)
+	)
+	(text "Flash"
+		(exclude_from_sim no)
+		(at 17.78 234.95 0)
+		(effects
+			(font
+				(size 2.54 2.54)
+			)
+			(justify left bottom)
+		)
+	)
+	(text "Clock Out\n"
+		(exclude_from_sim no)
+		(at 211.836 252.222 0)
+		(effects
+			(font
+				(size 2.54 2.54)
+			)
+			(justify left bottom)
+		)
+	)
+	(text "I2S DAC"
+		(exclude_from_sim no)
+		(at 306.832 35.56 0)
+		(effects
+			(font
+				(size 2.54 2.54)
+			)
+		)
+	)
+	(text "2.54mm Debug Connector"
+		(exclude_from_sim no)
+		(at 81.28 181.864 0)
+		(effects
+			(font
+				(size 1.27 1.27)
+			)
+			(justify left bottom)
+		)
+	)
+	(text "Make sure R7 and R8 are close to RP2350\n"
+		(exclude_from_sim no)
+		(at 261.62 129.54 0)
+		(effects
+			(font
+				(size 1.27 1.27)
+			)
+			(justify left bottom)
+		)
+	)
+	(text "Analog MUX"
+		(exclude_from_sim no)
+		(at 337.058 183.388 0)
+		(effects
+			(font
+				(size 2.54 2.54)
+			)
+			(justify left bottom)
+		)
+	)
+	(text "Gain select\nGSO GS1 Amp\nLow Low -6dB\nHigh Low 0dB\nLow High 3dB\nHigh High 6dB"
+		(exclude_from_sim no)
+		(at 139.954 74.422 0)
+		(effects
+			(font
+				(size 1.27 1.27)
+			)
+		)
+	)
+	(text "DVDD\n"
+		(exclude_from_sim no)
+		(at 323.596 25.4 0)
+		(effects
+			(font
+				(size 1.27 1.27)
+			)
+		)
+	)
+	(text "12MHz Crystal"
+		(exclude_from_sim no)
+		(at 27.94 135.89 0)
+		(effects
+			(font
+				(size 2.54 2.54)
+			)
+			(justify left bottom)
+		)
+	)
+	(text "Power"
+		(exclude_from_sim no)
+		(at 44.45 22.86 0)
+		(effects
+			(font
+				(size 2.54 2.54)
+			)
+			(justify left bottom)
+		)
+	)
 	(junction
 		(at 245.11 124.46)
@@
 		)
 	)
-	(circle
-		(center 142.24 135.255)
-		(radius 0.635)
-		(stroke
-			(width 0)
-			(type default)
-			(color 132 0 0 1)
-		)
-		(fill
-			(type color)
-			(color 132 0 0 1)
-		)
-	)
-	(text "CPVDD"
-		(exclude_from_sim no)
-		(at 386.842 24.384 0)
-		(effects
-			(font
-				(size 1.27 1.27)
-			)
-		)
-	)
-	(text "JST Debug Connector"
-		(exclude_from_sim no)
-		(at 37.465 183.515 0)
-		(effects
-			(font
-				(size 1.27 1.27)
-			)
-			(justify left bottom)
-		)
-	)
-	(text "For Opposite Side"
-		(exclude_from_sim no)
-		(at 90.678 62.23 0)
-		(effects
-			(font
-				(size 1.27 1.27)
-			)
-		)
-	)
-	(text "16 Pots"
-		(exclude_from_sim no)
-		(at 308.864 187.706 0)
-		(effects
-			(font
-				(size 2.54 2.54)
-			)
-			(justify left bottom)
-		)
-	)
-	(text "USB"
-		(exclude_from_sim no)
-		(at 18.542 85.852 0)
-		(effects
-			(font
-				(size 2.54 2.54)
-			)
-			(justify left bottom)
-		)
-	)
-	(text "Clock In\n"
-		(exclude_from_sim no)
-		(at 109.982 251.968 0)
-		(effects
-			(font
-				(size 2.54 2.54)
-			)
-			(justify left bottom)
-		)
-	)
-	(text "AMPLIFIER"
-		(exclude_from_sim no)
-		(at 177.546 27.432 0)
-		(effects
-			(font
-				(size 2.54 2.54)
-			)
-		)
-	)
-	(text "AVDD\n"
-		(exclude_from_sim no)
-		(at 349.758 24.638 0)
-		(effects
-			(font
-				(size 1.27 1.27)
-			)
-		)
-	)
-	(text "TODO: reduce the gain so it is safe for headphones?\nOr just trust that users will reduce volume from line level?"
-		(exclude_from_sim no)
-		(at 146.812 84.074 0)
-		(effects
-			(font
-				(size 1.27 1.27)
-			)
-		)
-	)
-	(text "Flash"
-		(exclude_from_sim no)
-		(at 17.78 234.95 0)
-		(effects
-			(font
-				(size 2.54 2.54)
-			)
-			(justify left bottom)
-		)
-	)
-	(text "Clock Out\n"
-		(exclude_from_sim no)
-		(at 211.836 252.222 0)
-		(effects
-			(font
-				(size 2.54 2.54)
-			)
-			(justify left bottom)
-		)
-	)
-	(text "I2S DAC"
-		(exclude_from_sim no)
-		(at 306.832 35.56 0)
-		(effects
-			(font
-				(size 2.54 2.54)
-			)
-		)
-	)
-	(text "2.54mm Debug Connector"
-		(exclude_from_sim no)
-		(at 81.28 181.864 0)
-		(effects
-			(font
-				(size 1.27 1.27)
-			)
-			(justify left bottom)
-		)
-	)
-	(text "Make sure R7 and R8 are close to RP2350\n"
-		(exclude_from_sim no)
-		(at 261.62 129.54 0)
-		(effects
-			(font
-				(size 1.27 1.27)
-			)
-			(justify left bottom)
-		)
-	)
-	(text "Analog MUX"
-		(exclude_from_sim no)
-		(at 337.058 183.388 0)
-		(effects
-			(font
-				(size 2.54 2.54)
-			)
-			(justify left bottom)
-		)
-	)
-	(text "Gain select\nGSO GS1 Amp\nLow Low -6dB\nHigh Low 0dB\nLow High 3dB\nHigh High 6dB"
-		(exclude_from_sim no)
-		(at 139.954 74.422 0)
-		(effects
-			(font
-				(size 1.27 1.27)
-			)
-		)
-	)
-	(text "DVDD\n"
-		(exclude_from_sim no)
-		(at 323.596 25.4 0)
-		(effects
-			(font
-				(size 1.27 1.27)
-			)
-		)
-	)
-	(text "12MHz Crystal"
-		(exclude_from_sim no)
-		(at 27.94 135.89 0)
-		(effects
-			(font
-				(size 2.54 2.54)
-			)
-			(justify left bottom)
-		)
-	)
-	(text "Power"
-		(exclude_from_sim no)
-		(at 44.45 22.86 0)
-		(effects
-			(font
-				(size 2.54 2.54)
-			)
-			(justify left bottom)
-		)
-	)
 	(label "P14"
 		(at 317.5 234.95 0)
@@
 			)
 		)
-		(property "LCSC" "C3010220"
+		(property "LCSC" "C782843"
 			(at 115.57 160.02 0)
 			(effects
@@
 			)
 		)
-		(property "LCSC" "C3010220"
+		(property "LCSC" "C782843"
 			(at 142.24 214.63 0)
 			(effects
@@
 		)
 	)
+	(embedded_fonts no)
 )
